File: KicadFiles/Tach/Tach Circuit.sch (KiCad schematic (older format))
At the start: 15 parts, among them Q1 2N3904

Commit message: ground = poured
Parts:
- added GND1: GND, Connector_PinHeader_2.54mm:PinHeader_1x02_P2.54mm_Vertical, symbol Connector:Conn_01x01_Female
- added VCC1: 5V, Connector_PinHeader_2.54mm:PinHeader_1x02_P2.54mm_Vertical, symbol Connector:Conn_01x01_Female
- D0, D1, D3: footprint Diode_THT:D_DO-41_SOD81_P10.16mm_Horizontal -> Diode_THT:D_DO-41_SOD81_P7.62mm_Horizontal
- D2: footprint Diode_THT:D_DO-35_SOD27_P7.62mm_Horizontal -> Diode_THT:D_T-1_P5.08mm_Horizontal
Connections:
- net +5V: now also VCC1.1 (Pin_1)
- net GND: now also GND1.1 (Pin_1)
Changed lines of the file:
@@
 F 0 "D0" V 2954 2729 50  0000 L CNN
 F 1 "1N4007" V 3045 2729 50  0000 L CNN
-F 2 "Diode_THT:D_DO-41_SOD81_P10.16mm_Horizontal" H 3000 2475 50  0001 C CNN
+F 2 "Diode_THT:D_DO-41_SOD81_P7.62mm_Horizontal" H 3000 2475 50  0001 C CNN
 F 3 "http://www.vishay.com/docs/88503/1n4001.pdf" H 3000 2650 50  0001 C CNN
 	1    3000 2650
@@
 F 0 "D1" H 3150 2284 50  0000 C CNN
 F 1 "1N4007" H 3150 2375 50  0000 C CNN
-F 2 "Diode_THT:D_DO-41_SOD81_P10.16mm_Horizontal" H 3150 2325 50  0001 C CNN
+F 2 "Diode_THT:D_DO-41_SOD81_P7.62mm_Horizontal" H 3150 2325 50  0001 C CNN
 F 3 "http://www.vishay.com/docs/88503/1n4001.pdf" H 3150 2500 50  0001 C CNN
 	1    3150 2500
@@
 F 0 "D2" H 3750 2284 50  0000 C CNN
 F 1 "1N4148" H 3750 2375 50  0000 C CNN
-F 2 "Diode_THT:D_DO-35_SOD27_P7.62mm_Horizontal" H 3750 2325 50  0001 C CNN
+F 2 "Diode_THT:D_T-1_P5.08mm_Horizontal" H 3750 2325 50  0001 C CNN
 F 3 "http://www.nxp.com/documents/data_sheet/1N4148_1N4448.pdf" H 3750 2500 50  0001 C CNN
 	1    3750 2500
@@
 F 0 "D3" V 3854 2729 50  0000 L CNN
 F 1 "1N4738" V 3945 2729 50  0000 L CNN
-F 2 "Diode_THT:D_DO-41_SOD81_P10.16mm_Horizontal" H 3900 2475 50  0001 C CNN
+F 2 "Diode_THT:D_DO-41_SOD81_P7.62mm_Horizontal" H 3900 2475 50  0001 C CNN
 F 3 "https://www.vishay.com/docs/85816/1n4728a.pdf" H 3900 2650 50  0001 C CNN
 	1    3900 2650
@@
 Wire Wire Line
 	5250 3550 4300 3550
+$Comp
+L Connector:Conn_01x01_Female VCC1
+U 1 1 5BC71D92
+P 4300 1800
+F 0 "VCC1" V 4238 1712 50  0000 R CNN
+F 1 "5V" V 4147 1712 50  0000 R CNN
+F 2 "Connector_PinHeader_2.54mm:PinHeader_1x02_P2.54mm_Vertical" H 4300 1800 50  0001 C CNN
+F 3 "~" H 4300 1800 50  0001 C CNN
+	1    4300 1800
+	0    -1   -1   0
+$EndComp
+$Comp
+L Connector:Conn_01x01_Female GND1
+U 1 1 5BC72FD8
+P 5900 3750
+F 0 "GND1" V 5746 3798 50  0000 L CNN
+F 1 "GND" V 5837 3798 50  0000 L CNN
+F 2 "Connector_PinHeader_2.54mm:PinHeader_1x02_P2.54mm_Vertical" H 5900 3750 50  0001 C CNN
+F 3 "~" H 5900 3750 50  0001 C CNN
+	1    5900 3750
+	0    1    1    0
+$EndComp
 $EndSCHEMATC
