File: KicadFiles/Backdash_v2/Backdash_v2.sch (KiCad schematic (older format))
At the start: 3 parts, among them J1 Conn_01x03_Female, J2 Conn_01x03_Female, J3 Conn_01x04_Female

Commit message: started back dash
Parts:
- added C? (x3): C, symbol Device:C
- added D?: D_Zener, symbol Device:D_Zener
- added L?: L, symbol Device:L
- added R? (x2): R, symbol Device:R
- added U?: TPS5430DDA, Package_SO:TI_SO-PowerPAD-8_ThermalVias, symbol Regulator_Switching:TPS5430DDA
Connections:
- net labels added: +BATT
- wire segments 6 -> 30
Other:
- note added: "REPLACE WITH TPS5410"
Changed lines of the file:
@@
 EESchema Schematic File Version 4
+LIBS:Backdash_v2-cache
 EELAYER 26 0
 EELAYER END
@@
 Text Notes 2700 1900 0    50   ~ 0
 OUTPUT FROM CVT TEMP
+$Comp
+L Regulator_Switching:TPS5430DDA U?
+U 1 1 5C0B6CD8
+P 2350 3850
+F 0 "U?" H 2350 4317 50  0000 C CNN
+F 1 "TPS5430DDA" H 2350 4226 50  0000 C CNN
+F 2 "Package_SO:TI_SO-PowerPAD-8_ThermalVias" H 2400 3500 50  0001 L CIN
+F 3 "http://www.ti.com/lit/ds/symlink/tps5430.pdf" H 2350 3850 50  0001 C CNN
+	1    2350 3850
+	1    0    0    -1
+$EndComp
+Text Notes 1900 3350 0    50   ~ 0
+REPLACE WITH TPS5410
+$Comp
+L power:+BATT #PWR?
+U 1 1 5C0B6DAC
+P 1550 3600
+F 0 "#PWR?" H 1550 3450 50  0001 C CNN
+F 1 "+BATT" H 1565 3773 50  0000 C CNN
+F 2 "" H 1550 3600 50  0001 C CNN
+F 3 "" H 1550 3600 50  0001 C CNN
+	1    1550 3600
+	1    0    0    -1
+$EndComp
+$Comp
+L power:GND #PWR?
+U 1 1 5C0B6E4E
+P 2250 4300
+F 0 "#PWR?" H 2250 4050 50  0001 C CNN
+F 1 "GND" H 2255 4127 50  0000 C CNN
+F 2 "" H 2250 4300 50  0001 C CNN
+F 3 "" H 2250 4300 50  0001 C CNN
+	1    2250 4300
+	1    0    0    -1
+$EndComp
+Wire Wire Line
+	2250 4300 2250 4250
+Wire Wire Line
+	1850 3650 1650 3650
+Wire Wire Line
+	1550 3650 1550 3600
+Wire Wire Line
+	1850 4050 1650 4050
+Wire Wire Line
+	1650 4050 1650 3650
+Connection ~ 1650 3650
+Wire Wire Line
+	1650 3650 1550 3650
+$Comp
+L Device:C C?
+U 1 1 5C0B72DC
+P 3200 3800
+F 0 "C?" H 3315 3846 50  0000 L CNN
+F 1 "C" H 3315 3755 50  0000 L CNN
+F 2 "" H 3238 3650 50  0001 C CNN
+F 3 "~" H 3200 3800 50  0001 C CNN
+	1    3200 3800
+	1    0    0    -1
+$EndComp
+Wire Wire Line
+	2850 3650 3200 3650
+$Comp
+L Device:L L?
+U 1 1 5C0B7712
+P 3650 3650
+F 0 "L?" V 3840 3650 50  0000 C CNN
+F 1 "L" V 3749 3650 50  0000 C CNN
+F 2 "" H 3650 3650 50  0001 C CNN
+F 3 "~" H 3650 3650 50  0001 C CNN
+	1    3650 3650
+	0    -1   -1   0
+$EndComp
+$Comp
+L Device:C C?
+U 1 1 5C0B777B
+P 4000 3800
+F 0 "C?" H 4115 3846 50  0000 L CNN
+F 1 "C" H 4115 3755 50  0000 L CNN
+F 2 "" H 4038 3650 50  0001 C CNN
+F 3 "~" H 4000 3800 50  0001 C CNN
+	1    4000 3800
+	1    0    0    -1
+$EndComp
+$Comp
+L Device:R R?
+U 1 1 5C0B77CF
+P 4500 3750
+F 0 "R?" H 4570 3796 50  0000 L CNN
+F 1 "R" H 4570 3705 50  0000 L CNN
+F 2 "" V 4430 3750 50  0001 C CNN
+F 3 "~" H 4500 3750 50  0001 C CNN
+	1    4500 3750
+	1    0    0    -1
+$EndComp
+$Comp
+L Device:R R?
+U 1 1 5C0B7825
+P 4500 4200
+F 0 "R?" H 4570 4246 50  0000 L CNN
+F 1 "R" H 4570 4155 50  0000 L CNN
+F 2 "" V 4430 4200 50  0001 C CNN
+F 3 "~" H 4500 4200 50  0001 C CNN
+	1    4500 4200
+	1    0    0    -1
+$EndComp
+$Comp
+L power:GND #PWR?
+U 1 1 5C0B785D
+P 4500 4350
+F 0 "#PWR?" H 4500 4100 50  0001 C CNN
+F 1 "GND" H 4505 4177 50  0000 C CNN
+F 2 "" H 4500 4350 50  0001 C CNN
+F 3 "" H 4500 4350 50  0001 C CNN
+	1    4500 4350
+	1    0    0    -1
+$EndComp
+Wire Wire Line
+	2250 4250 2350 4250
+Connection ~ 2250 4250
+Wire Wire Line
+	4500 4050 4500 4000
+Wire Wire Line
+	4500 4000 4350 4000
+Wire Wire Line
+	4350 4000 4350 4050
+Wire Wire Line
+	4350 4050 2850 4050
+Connection ~ 4500 4000
+Wire Wire Line
+	4500 4000 4500 3900
+Wire Wire Line
+	3800 3650 4000 3650
+Wire Wire Line
+	4000 3650 4300 3650
+Wire Wire Line
+	4300 3650 4300 3600
+Wire Wire Line
+	4300 3600 4500 3600
+Connection ~ 4000 3650
+Wire Wire Line
+	4500 3600 4900 3600
+Connection ~ 4500 3600
+$Comp
+L power:+5V #PWR?
+U 1 1 5C0B8C40
+P 4900 3600
+F 0 "#PWR?" H 4900 3450 50  0001 C CNN
+F 1 "+5V" H 4915 3773 50  0000 C CNN
+F 2 "" H 4900 3600 50  0001 C CNN
+F 3 "" H 4900 3600 50  0001 C CNN
+	1    4900 3600
+	1    0    0    -1
+$EndComp
+$Comp
+L power:GND #PWR?
+U 1 1 5C0B8CB5
+P 4000 3950
+F 0 "#PWR?" H 4000 3700 50  0001 C CNN
+F 1 "GND" H 4005 3777 50  0000 C CNN
+F 2 "" H 4000 3950 50  0001 C CNN
+F 3 "" H 4000 3950 50  0001 C CNN
+	1    4000 3950
+	1    0    0    -1
+$EndComp
+$Comp
+L Device:C C?
+U 1 1 5C0B8DB4
+P 1400 3850
+F 0 "C?" H 1515 3896 50  0000 L CNN
+F 1 "C" H 1515 3805 50  0000 L CNN
+F 2 "" H 1438 3700 50  0001 C CNN
+F 3 "~" H 1400 3850 50  0001 C CNN
+	1    1400 3850
+	1    0    0    -1
+$EndComp
+$Comp
+L power:GND #PWR?
+U 1 1 5C0B8E1A
+P 1400 4000
+F 0 "#PWR?" H 1400 3750 50  0001 C CNN
+F 1 "GND" H 1405 3827 50  0000 C CNN
+F 2 "" H 1400 4000 50  0001 C CNN
+F 3 "" H 1400 4000 50  0001 C CNN
+	1    1400 4000
+	1    0    0    -1
+$EndComp
+Wire Wire Line
+	1400 3700 1400 3650
+Wire Wire Line
+	1400 3650 1550 3650
+Connection ~ 1550 3650
+$Comp
+L Device:D_Zener D?
+U 1 1 5C0B92FF
+P 3450 3800
+F 0 "D?" V 3404 3879 50  0000 L CNN
+F 1 "D_Zener" V 3495 3879 50  0000 L CNN
+F 2 "" H 3450 3800 50  0001 C CNN
+F 3 "~" H 3450 3800 50  0001 C CNN
+	1    3450 3800
+	0    1    1    0
+$EndComp
+Connection ~ 3450 3650
+Wire Wire Line
+	3450 3650 3500 3650
+Wire Wire Line
+	3200 3650 3450 3650
+Connection ~ 3200 3650
+$Comp
+L power:GND #PWR?
+U 1 1 5C0B99BA
+P 3450 3950
+F 0 "#PWR?" H 3450 3700 50  0001 C CNN
+F 1 "GND" H 3455 3777 50  0000 C CNN
+F 2 "" H 3450 3950 50  0001 C CNN
+F 3 "" H 3450 3950 50  0001 C CNN
+	1    3450 3950
+	1    0    0    -1
+$EndComp
+Wire Wire Line
+	2850 3950 2850 3850
+Wire Wire Line
+	2850 3950 3200 3950
 $EndSCHEMATC
