File: KicadFiles/FrontDash_circuitry/FrontDash_circuitry.sch (KiCad schematic (older format))
At the start: 6 parts, among them U1 DS3231M

Commit message: Starting ATMEGA
Parts:
- added C? (x2): C, symbol Device:C
- added U?: ATmega328P-AU, Package_QFP:TQFP-32_7x7mm_P0.8mm, symbol MCU_Microchip_ATmega:ATmega328P-AU
- added Y?: Crystal, symbol Device:Crystal
Connections:
- net labels added: XTAL1, XTAL2
- wire segments 10 -> 18
Changed lines of the file:
@@
 EESchema Schematic File Version 4
-EELAYER 26 0
+LIBS:FrontDash_circuitry-cache
+EELAYER 28 0
 EELAYER END
 $Descr A4 11693 8268
@@
 	1    0    0    -1
 $EndComp
+$Comp
+L MCU_Microchip_ATmega:ATmega328P-AU U?
+U 1 1 5BEB9259
+P 2400 5500
+F 0 "U?" H 1550 4200 50  0000 C CNN
+F 1 "ATmega328P-AU" H 1500 4150 50  0000 C CNN
+F 2 "Package_QFP:TQFP-32_7x7mm_P0.8mm" H 2400 5500 50  0001 C CIN
+F 3 "http://ww1.microchip.com/downloads/en/DeviceDoc/ATmega328_P%20AVR%20MCU%20with%20picoPower%20Technology%20Data%20Sheet%2040001984A.pdf" H 2400 5500 50  0001 C CNN
+	1    2400 5500
+	1    0    0    -1
+$EndComp
+$Comp
+L Device:Crystal Y?
+U 1 1 5BEBC3A0
+P 3600 4950
+F 0 "Y?" V 3554 5081 50  0000 L CNN
+F 1 "Crystal" V 3645 5081 50  0000 L CNN
+F 2 "" H 3600 4950 50  0001 C CNN
+F 3 "~" H 3600 4950 50  0001 C CNN
+	1    3600 4950
+	0    1    1    0
+$EndComp
+$Comp
+L Device:C C?
+U 1 1 5BEBCC31
+P 4150 4800
+F 0 "C?" V 3898 4800 50  0000 C CNN
+F 1 "C" V 3989 4800 50  0000 C CNN
+F 2 "" H 4188 4650 50  0001 C CNN
+F 3 "~" H 4150 4800 50  0001 C CNN
+	1    4150 4800
+	0    1    1    0
+$EndComp
+$Comp
+L Device:C C?
+U 1 1 5BEBE28E
+P 4150 5100
+F 0 "C?" V 3898 5100 50  0000 C CNN
+F 1 "C" V 3989 5100 50  0000 C CNN
+F 2 "" H 4188 4950 50  0001 C CNN
+F 3 "~" H 4150 5100 50  0001 C CNN
+	1    4150 5100
+	0    1    1    0
+$EndComp
+Wire Wire Line
+	3450 4800 3600 4800
+Text Label 3000 4900 0    50   ~ 0
+XTAL1
+Text Label 3000 5000 0    50   ~ 0
+XTAL2
+Text Label 3450 4800 0    50   ~ 0
+XTAL1
+Wire Wire Line
+	3450 5100 3600 5100
+Text Label 3450 5100 0    50   ~ 0
+XTAL2
+Wire Wire Line
+	3600 4800 4000 4800
+Connection ~ 3600 4800
+Wire Wire Line
+	3600 5100 4000 5100
+Connection ~ 3600 5100
+$Comp
+L power:GND #PWR?
+U 1 1 5BEC73B8
+P 4550 5100
+F 0 "#PWR?" H 4550 4850 50  0001 C CNN
+F 1 "GND" H 4555 4927 50  0000 C CNN
+F 2 "" H 4550 5100 50  0001 C CNN
+F 3 "" H 4550 5100 50  0001 C CNN
+	1    4550 5100
+	1    0    0    -1
+$EndComp
+Wire Wire Line
+	4300 4800 4300 4950
+Wire Wire Line
+	4550 4950 4300 4950
+Wire Wire Line
+	4550 5100 4550 4950
+Connection ~ 4300 4950
+Wire Wire Line
+	4300 4950 4300 5100
+$Comp
+L power:GND #PWR?
+U 1 1 5BECAC8B
+P 2400 7000
+F 0 "#PWR?" H 2400 6750 50  0001 C CNN
+F 1 "GND" H 2405 6827 50  0000 C CNN
+F 2 "" H 2400 7000 50  0001 C CNN
+F 3 "" H 2400 7000 50  0001 C CNN
+	1    2400 7000
+	1    0    0    -1
+$EndComp
+Wire Bus Line
+	550  7750 6900 7750
+Wire Bus Line
+	6900 3350 550  3350
+Wire Bus Line
+	550  3350 550  7750
+Wire Bus Line
+	6900 3350 6900 7750
 $EndSCHEMATC

Commit message: nano progress made
Parts:
- added C4, C5, C6: 100n, symbol Device:C
- added D?: LED, symbol Device:LED
- added J1: ICSP, symbol Connector_Generic:Conn_02x03_Counter_Clockwise
- added R5, R6: 1k, symbol Device:R
- added SW1: SW_Push, symbol Switch:SW_Push
- C2, C3: renamed from C?; value C -> 22p
Connections:
- net labels added: +5V, A0, A1, A2, A3, A4, A5, A6, A7, AREF, AVCC, D10, D2, D3, D4, D5, D6, D7, D8, D9, MISO, MOSI, RESET, RX, TX, VCC
- wire segments 18 -> 29
Other:
- moved on the sheet: C2, C3, Y?

Commit message: Added can circuitry
Parts:
- added C7, C?: 100 nF, symbol Device:C
- added C? (x2): 22pF, symbol Device:C
- added J2, J3: Conn_01x02_Male, symbol Connector:Conn_01x02_Male
- added J? (x2): Conn_01x08_Male, symbol Connector:Conn_01x08_Male
- added R5: 10 ohm, symbol Device:R
- added R6: 120, symbol Device:R
- added R? (x2): 100K, symbol Device:R
- added U4: MCP2551-I-P, Package_DIP:DIP-8_W7.62mm, symbol Interface_CAN_LIN:MCP2551-I-P
- added Y1: 10MHz, symbol Device:Crystal
- U1: renamed from U?; symbol MCU_Microchip_ATmega:ATmega328P-AU -> FrontDash_circuitry-rescue:ATmega328P-AU-MCU_Microchip_ATmega
- gave numbers to parts that had none: 3
- renumbered C5 to C1, C4 to C2, C2 to C3, C3 to C4, C6 to C5, C1 to C6, R6 to R1, R4 to R2, R5 to R3, R3 to R4, U1 to U2
Connections:
- net labels added: INT
- wire segments 29 -> 71
Other:
- note added: "CAN CONTROLLER"
- note added: "CAN TRANSCEIVER"
- note added: "CAN system: Transceiver and Controller"
- note added: "JUMPER"
- note added: "MINI SD CARD \nhttps://learn.adafruit.com/adafruit-micro-sd-breakout-board-card-tutorial/download"
- note added: "NC"
- note added: "NC\nNC"
- note added: "RTC"
- note added: "https://download.mikroe.com/documents/add-on-boards/click/canspi-5v/can-spi-click-5v-manual-v100.pdf"
- moved on the sheet: U3

Commit message: nano completed
Parts:
- added C?: 1u, symbol Device:C
- added C?: 4.7u, symbol Device:CP
- C2: value 100n -> 1u
Connections:
- net +5V: now also C?.1, C?.1
- net GND: now also C?.2, C?.2
Other:
- note added: "AtMega 328p (nano)\n"
- moved on the sheet: C2, SW1
Changed lines of the file:
@@
 EESchema Schematic File Version 4
 LIBS:FrontDash_circuitry-cache
-EELAYER 26 0
+EELAYER 28 0
 EELAYER END
 $Descr A4 11693 8268
@@
 Wire Wire Line
 	1450 3800 1450 3950
-Wire Bus Line
-	550  7750 6900 7750
-Wire Bus Line
-	6900 3350 550  3350
-Wire Bus Line
-	550  3350 550  7750
-Wire Bus Line
-	6900 3350 6900 7750
 Text Label 2400 4000 1    50   ~ 0
 VCC
@@
 AVCC
 Wire Wire Line
-	800  4400 950  4400
-Text Label 1100 4400 0    50   ~ 0
+	3600 4300 3750 4300
+Text Label 3900 4300 0    50   ~ 0
 AVCC
-Text Label 800  4400 2    50   ~ 0
+Text Label 3600 4300 2    50   ~ 0
 VCC
 $Comp
 L Device:C C2
 U 1 1 5BEEEC4C
-P 950 4550
-F 0 "C2" H 1065 4596 50  0000 L CNN
-F 1 "100n" H 1065 4505 50  0000 L CNN
-F 2 "" H 988 4400 50  0001 C CNN
-F 3 "~" H 950 4550 50  0001 C CNN
-	1    950  4550
+P 4100 4750
+F 0 "C2" H 4215 4796 50  0000 L CNN
+F 1 "1u" H 4215 4705 50  0000 L CNN
+F 2 "" H 4138 4600 50  0001 C CNN
+F 3 "~" H 4100 4750 50  0001 C CNN
+	1    4100 4750
 	1    0    0    -1
 $EndComp
@@
 	1    0    0    -1
 $EndComp
-Connection ~ 950  4400
-Wire Wire Line
-	950  4300 950  4400
-Wire Wire Line
-	1100 4400 950  4400
+Connection ~ 3750 4300
+Wire Wire Line
+	3750 4200 3750 4300
+Wire Wire Line
+	3900 4300 3750 4300
 Text Label 3000 5800 0    50   ~ 0
 RESET
@@
 L Switch:SW_Push SW1
 U 1 1 5BF1B5B4
-P 900 5050
-F 0 "SW1" H 900 5335 50  0000 C CNN
-F 1 "SW_Push" H 900 5244 50  0000 C CNN
-F 2 "" H 900 5250 50  0001 C CNN
-F 3 "" H 900 5250 50  0001 C CNN
-	1    900  5050
+P 1000 4750
+F 0 "SW1" H 1000 5035 50  0000 C CNN
+F 1 "SW_Push" H 1000 4944 50  0000 C CNN
+F 2 "" H 1000 4950 50  0001 C CNN
+F 3 "" H 1000 4950 50  0001 C CNN
+	1    1000 4750
 	0    -1   -1   0
 $EndComp
@@
 Wire Wire Line
 	1600 5200 1200 5200
-Text Label 950  4700 0    50   ~ 0
+Text Label 3750 5300 0    50   ~ 0
 GND
 Text Label 2400 7000 0    50   ~ 0
@@
 	1    0    0    -1
 $EndComp
-Text Label 900  4850 0    50   ~ 0
+Text Label 1000 4550 0    50   ~ 0
 RESET
-Text Label 900  5250 0    50   ~ 0
+Text Label 1000 4950 0    50   ~ 0
 GND
 Text Label 1200 4800 0    50   ~ 0
@@
 Text Label 3700 3800 2    50   ~ 0
 SCK
-Text Label 950  4300 0    50   ~ 0
+Text Label 3750 4200 0    50   ~ 0
 +5V
 Text Label 700  5400 0    50   ~ 0
@@
 Text Notes 7450 4200 0    59   ~ 0
 RTC
+$Comp
+L Device:C C?
+U 1 1 5C01A2F6
+P 3350 4750
+F 0 "C?" H 3465 4796 50  0000 L CNN
+F 1 "1u" H 3465 4705 50  0000 L CNN
+F 2 "" H 3388 4600 50  0001 C CNN
+F 3 "~" H 3350 4750 50  0001 C CNN
+	1    3350 4750
+	1    0    0    -1
+$EndComp
+$Comp
+L Device:CP C?
+U 1 1 5C023C80
+P 3750 4750
+F 0 "C?" H 3868 4796 50  0000 L CNN
+F 1 "4.7u" H 3868 4705 50  0000 L CNN
+F 2 "" H 3788 4600 50  0001 C CNN
+F 3 "~" H 3750 4750 50  0001 C CNN
+	1    3750 4750
+	1    0    0    -1
+$EndComp
+Wire Wire Line
+	3750 4300 3750 4450
+Wire Wire Line
+	3350 4600 3350 4450
+Wire Wire Line
+	3350 4450 3750 4450
+Connection ~ 3750 4450
+Wire Wire Line
+	3750 4450 3750 4600
+Wire Wire Line
+	3750 4450 4100 4450
+Wire Wire Line
+	4100 4450 4100 4600
+Wire Wire Line
+	4100 4900 4100 5100
+Wire Wire Line
+	4100 5100 3750 5100
+Wire Wire Line
+	3350 5100 3350 4900
+Wire Wire Line
+	3750 4900 3750 5100
+Connection ~ 3750 5100
+Wire Wire Line
+	3750 5100 3350 5100
+Wire Wire Line
+	3750 5100 3750 5300
+Text Notes 3350 7450 0    50   ~ 0
+AtMega 328p (nano)\n
+Wire Notes Line
+	550  7650 4450 7650
+Wire Notes Line
+	4450 7650 4450 3300
+Wire Notes Line
+	4450 3300 550  3300
+Wire Notes Line
+	550  3300 550  7650
 $EndSCHEMATC

Commit message: Front dash mini sd card is almost done
Parts:
- added C? (x2): 100 nF, symbol Device:C
- added J?: Micro_SD_Card, symbol Connector:Micro_SD_Card
- added U?: LP2985-3.3, Package_TO_SOT_SMD:SOT-23-5, symbol Regulator_Linear:LP2985-3.3
Connections:
- net labels added: CD_SD, CLK
- wire segments 83 -> 99
Other:
- note added: "Linear Regulator"
- note added: "https://learn.adafruit.com/assets/35635"
- note added: "insert CD54HC4050 here (level shifter)"
- note removed: "RTC"
Changed lines of the file:
@@
 EESchema Schematic File Version 4
 LIBS:FrontDash_circuitry-cache
-EELAYER 28 0
+EELAYER 26 0
 EELAYER END
 $Descr A4 11693 8268
@@
 Text Notes 7400 4050 0    59   ~ 0
 MINI SD CARD \nhttps://learn.adafruit.com/adafruit-micro-sd-breakout-board-card-tutorial/download
-Text Notes 7450 4200 0    59   ~ 0
-RTC
 $Comp
 L Device:C C?
@@
 Wire Notes Line
 	550  3300 550  7650
+$Comp
+L Regulator_Linear:LP2985-3.3 U?
+U 1 1 5C075051
+P 6050 3900
+F 0 "U?" H 6050 4242 50  0000 C CNN
+F 1 "LP2985-3.3" H 6050 4151 50  0000 C CNN
+F 2 "Package_TO_SOT_SMD:SOT-23-5" H 6050 4225 50  0001 C CNN
+F 3 "http://www.ti.com/lit/ds/symlink/lp2985.pdf" H 6050 3900 50  0001 C CNN
+	1    6050 3900
+	1    0    0    -1
+$EndComp
+$Comp
+L power:+3V3 #PWR?
+U 1 1 5C0753B8
+P 6550 3750
+F 0 "#PWR?" H 6550 3600 50  0001 C CNN
+F 1 "+3V3" H 6565 3923 50  0000 C CNN
+F 2 "" H 6550 3750 50  0001 C CNN
+F 3 "" H 6550 3750 50  0001 C CNN
+	1    6550 3750
+	1    0    0    -1
+$EndComp
+Wire Wire Line
+	6450 3800 6550 3800
+Wire Wire Line
+	6550 3800 6550 3750
+$Comp
+L power:GND #PWR?
+U 1 1 5C0774A6
+P 6050 4200
+F 0 "#PWR?" H 6050 3950 50  0001 C CNN
+F 1 "GND" H 6055 4027 50  0000 C CNN
+F 2 "" H 6050 4200 50  0001 C CNN
+F 3 "" H 6050 4200 50  0001 C CNN
+	1    6050 4200
+	1    0    0    -1
+$EndComp
+$Comp
+L power:+5V #PWR?
+U 1 1 5C0779E3
+P 5550 3800
+F 0 "#PWR?" H 5550 3650 50  0001 C CNN
+F 1 "+5V" H 5565 3973 50  0000 C CNN
+F 2 "" H 5550 3800 50  0001 C CNN
+F 3 "" H 5550 3800 50  0001 C CNN
+	1    5550 3800
+	1    0    0    -1
+$EndComp
+Wire Wire Line
+	5650 3800 5550 3800
+$Comp
+L Device:C C?
+U 1 1 5C079EC3
+P 6800 3950
+F 0 "C?" H 6915 3996 50  0000 L CNN
+F 1 "100 nF" H 6915 3905 50  0000 L CNN
+F 2 "" H 6838 3800 50  0001 C CNN
+F 3 "~" H 6800 3950 50  0001 C CNN
+	1    6800 3950
+	1    0    0    -1
+$EndComp
+$Comp
+L Device:C C?
+U 1 1 5C07A03B
+P 5100 3950
+F 0 "C?" H 5215 3996 50  0000 L CNN
+F 1 "100 nF" H 5215 3905 50  0000 L CNN
+F 2 "" H 5138 3800 50  0001 C CNN
+F 3 "~" H 5100 3950 50  0001 C CNN
+	1    5100 3950
+	1    0    0    -1
+$EndComp
+Wire Wire Line
+	5550 3800 5500 3800
+Connection ~ 5550 3800
+Wire Wire Line
+	6550 3800 6800 3800
+Connection ~ 6550 3800
+$Comp
+L power:GND #PWR?
+U 1 1 5C07E085
+P 5100 4100
+F 0 "#PWR?" H 5100 3850 50  0001 C CNN
+F 1 "GND" H 5105 3927 50  0000 C CNN
+F 2 "" H 5100 4100 50  0001 C CNN
+F 3 "" H 5100 4100 50  0001 C CNN
+	1    5100 4100
+	1    0    0    -1
+$EndComp
+$Comp
+L power:GND #PWR?
+U 1 1 5C07E0DA
+P 6800 4100
+F 0 "#PWR?" H 6800 3850 50  0001 C CNN
+F 1 "GND" H 6805 3927 50  0000 C CNN
+F 2 "" H 6800 4100 50  0001 C CNN
+F 3 "" H 6800 4100 50  0001 C CNN
+	1    6800 4100
+	1    0    0    -1
+$EndComp
+Wire Wire Line
+	5650 3900 5500 3900
+Wire Wire Line
+	5500 3900 5500 3800
+Connection ~ 5500 3800
+Wire Wire Line
+	5500 3800 5100 3800
+Text Notes 5250 3550 0    50   ~ 0
+Linear Regulator
+Wire Notes Line
+	4600 3300 11050 3300
+Wire Notes Line
+	11050 3300 11050 6450
+Wire Notes Line
+	11050 6450 4600 6450
+Wire Notes Line
+	4600 6450 4600 3300
+Text Notes 5700 5650 0    50   ~ 0
+insert CD54HC4050 here (level shifter)
+$Comp
+L Connector:Micro_SD_Card J?
+U 1 1 5C085268
+P 8600 5450
+F 0 "J?" H 8550 6167 50  0000 C CNN
+F 1 "Micro_SD_Card" H 8550 6076 50  0000 C CNN
+F 2 "" H 9750 5750 50  0001 C CNN
+F 3 "http://katalog.we-online.de/em/datasheet/693072010801.pdf" H 8600 5450 50  0001 C CNN
+	1    8600 5450
+	1    0    0    -1
+$EndComp
+$Comp
+L power:GND #PWR?
+U 1 1 5C0855B0
+P 9400 6050
+F 0 "#PWR?" H 9400 5800 50  0001 C CNN
+F 1 "GND" H 9405 5877 50  0000 C CNN
+F 2 "" H 9400 6050 50  0001 C CNN
+F 3 "" H 9400 6050 50  0001 C CNN
+	1    9400 6050
+	1    0    0    -1
+$EndComp
+Wire Wire Line
+	7700 5650 7550 5650
+Wire Wire Line
+	7700 5550 7300 5550
+Wire Wire Line
+	7300 5450 7700 5450
+Wire Wire Line
+	7700 5350 7300 5350
+Wire Wire Line
+	7300 5250 7700 5250
+Wire Wire Line
+	7700 5150 7300 5150
+Wire Wire Line
+	7300 5750 7700 5750
+Wire Wire Line
+	7300 5850 7700 5850
+$Comp
+L power:GND #PWR?
+U 1 1 5C0B5CF7
+P 7550 5650
+F 0 "#PWR?" H 7550 5400 50  0001 C CNN
+F 1 "GND" H 7555 5477 50  0000 C CNN
+F 2 "" H 7550 5650 50  0001 C CNN
+F 3 "" H 7550 5650 50  0001 C CNN
+	1    7550 5650
+	0    1    1    0
+$EndComp
+$Comp
+L power:+3V3 #PWR?
+U 1 1 5C0B5E0C
+P 7300 5450
+F 0 "#PWR?" H 7300 5300 50  0001 C CNN
+F 1 "+3V3" H 7315 5623 50  0000 C CNN
+F 2 "" H 7300 5450 50  0001 C CNN
+F 3 "" H 7300 5450 50  0001 C CNN
+	1    7300 5450
+	0    -1   -1   0
+$EndComp
+Text Label 7300 5550 0    50   ~ 0
+CLK
+Text Label 7300 5250 0    50   ~ 0
+CD_SD
+Text Notes 6050 4950 0    50   ~ 0
+https://learn.adafruit.com/assets/35635
 $EndSCHEMATC

Commit message: started back dash
Parts:
- R1, R3: footprint (none) -> Resistor_THT:R_Axial_DIN0207_L6.3mm_D2.5mm_P7.62mm_Horizontal
- gave numbers to parts that had none: 13
- renumbered Y1 to Y2
Changed lines of the file:
@@
 F 0 "R3" H 1670 4996 50  0000 L CNN
 F 1 "1k" H 1670 4905 50  0000 L CNN
-F 2 "" V 1530 4950 50  0001 C CNN
+F 2 "Resistor_THT:R_Axial_DIN0207_L6.3mm_D2.5mm_P7.62mm_Horizontal" V 1530 4950 50  0001 C CNN
 F 3 "~" H 1600 4950 50  0001 C CNN
 	1    1600 4950
@@
 F 0 "R1" V 743 5500 50  0000 C CNN
 F 1 "1k" V 834 5500 50  0000 C CNN
-F 2 "" V 880 5500 50  0001 C CNN
+F 2 "Resistor_THT:R_Axial_DIN0207_L6.3mm_D2.5mm_P7.62mm_Horizontal" V 880 5500 50  0001 C CNN
 F 3 "~" H 950 5500 50  0001 C CNN
 	1    950  5500
@@
 $EndComp
 $Comp
-L Device:C C?
+L Device:C C14
 U 1 1 5BFEB36C
 P 6900 1000
-F 0 "C?" H 7015 1046 50  0000 L CNN
+F 0 "C14" H 7015 1046 50  0000 L CNN
 F 1 "100 nF" H 7015 955 50  0000 L CNN
 F 2 "" H 6938 850 50  0001 C CNN
@@
 Connection ~ 9700 850
 $Comp
-L power:GND #PWR?
+L power:GND #PWR027
 U 1 1 5BFEC5D3
 P 8950 1150
-F 0 "#PWR?" H 8950 900 50  0001 C CNN
+F 0 "#PWR027" H 8950 900 50  0001 C CNN
 F 1 "GND" H 8955 977 50  0000 C CNN
 F 2 "" H 8950 1150 50  0001 C CNN
@@
 $EndComp
 $Comp
-L power:+5V #PWR?
+L power:+5V #PWR026
 U 1 1 5BFEC642
 P 7800 850
-F 0 "#PWR?" H 7800 700 50  0001 C CNN
+F 0 "#PWR026" H 7800 700 50  0001 C CNN
 F 1 "+5V" H 7815 1023 50  0000 C CNN
 F 2 "" H 7800 850 50  0001 C CNN
@@
 Connection ~ 7800 850
 $Comp
-L power:GND #PWR?
+L power:GND #PWR023
 U 1 1 5BFED8C3
 P 6900 1150
-F 0 "#PWR?" H 6900 900 50  0001 C CNN
+F 0 "#PWR023" H 6900 900 50  0001 C CNN
 F 1 "GND" H 6905 977 50  0000 C CNN
 F 2 "" H 6900 1150 50  0001 C CNN
@@
 	6900 850  7800 850
 $Comp
-L Device:Crystal Y1
+L Device:Crystal Y2
 U 1 1 5BFEE61E
 P 6450 2300
-F 0 "Y1" H 6450 2568 50  0000 C CNN
+F 0 "Y2" H 6450 2568 50  0000 C CNN
 F 1 "10MHz" H 6450 2477 50  0000 C CNN
 F 2 "" H 6450 2300 50  0001 C CNN
@@
 	6200 2300 6300 2300
 $Comp
-L Device:C C?
+L Device:C C11
 U 1 1 5BFEFE89
 P 6200 2550
-F 0 "C?" H 6315 2596 50  0000 L CNN
+F 0 "C11" H 6315 2596 50  0000 L CNN
 F 1 "22pF" H 6315 2505 50  0000 L CNN
 F 2 "" H 6238 2400 50  0001 C CNN
@@
 $EndComp
 $Comp
-L Device:C C?
+L Device:C C12
 U 1 1 5BFEFEE9
 P 6650 2550
-F 0 "C?" H 6765 2596 50  0000 L CNN
+F 0 "C12" H 6765 2596 50  0000 L CNN
 F 1 "22pF" H 6765 2505 50  0000 L CNN
 F 2 "" H 6688 2400 50  0001 C CNN
@@
 	6650 2300 7200 2300
 $Comp
-L power:GND #PWR?
+L power:GND #PWR021
 U 1 1 5BFF1722
 P 6650 2700
-F 0 "#PWR?" H 6650 2450 50  0001 C CNN
+F 0 "#PWR021" H 6650 2450 50  0001 C CNN
 F 1 "GND" H 6655 2527 50  0000 C CNN
 F 2 "" H 6650 2700 50  0001 C CNN
@@
 $EndComp
 $Comp
-L power:GND #PWR?
+L power:GND #PWR019
 U 1 1 5BFF1765
 P 6200 2700
-F 0 "#PWR?" H 6200 2450 50  0001 C CNN
+F 0 "#PWR019" H 6200 2450 50  0001 C CNN
 F 1 "GND" H 6205 2527 50  0000 C CNN
 F 2 "" H 6200 2700 50  0001 C CNN
@@
 $EndComp
 $Comp
-L Device:R R?
+L Device:R R7
 U 1 1 5BFF1C24
 P 8700 2800
-F 0 "R?" V 8907 2800 50  0000 C CNN
+F 0 "R7" V 8907 2800 50  0000 C CNN
 F 1 "100K" V 8816 2800 50  0000 C CNN
 F 2 "" V 8630 2800 50  0001 C CNN
@@
 	8400 2800 8400 2600
 $Comp
-L power:+5V #PWR?
+L power:+5V #PWR028
 U 1 1 5BFF2AAC
 P 8950 2750
-F 0 "#PWR?" H 8950 2600 50  0001 C CNN
+F 0 "#PWR028" H 8950 2600 50  0001 C CNN
 F 1 "+5V" H 8965 2923 50  0000 C CNN
 F 2 "" H 8950 2750 50  0001 C CNN
@@
 	8550 2400 8550 2300
 $Comp
-L Device:R R?
+L Device:R R8
 U 1 1 5BFF5C73
 P 8750 2300
-F 0 "R?" V 8957 2300 50  0000 C CNN
+F 0 "R8" V 8957 2300 50  0000 C CNN
 F 1 "100K" V 8866 2300 50  0000 C CNN
 F 2 "" V 8680 2300 50  0001 C CNN
@@
 $EndComp
 $Comp
-L power:+5V #PWR?
+L power:+5V #PWR029
 U 1 1 5BFF5CC5
 P 9000 2250
-F 0 "#PWR?" H 9000 2100 50  0001 C CNN
+F 0 "#PWR029" H 9000 2100 50  0001 C CNN
 F 1 "+5V" H 9015 2423 50  0000 C CNN
 F 2 "" H 9000 2250 50  0001 C CNN
@@
 NC
 $Comp
-L Connector:Conn_01x08_Male J?
+L Connector:Conn_01x08_Male J5
 U 1 1 5BFFAFB3
 P 5600 1700
-F 0 "J?" H 5706 2178 50  0000 C CNN
+F 0 "J5" H 5706 2178 50  0000 C CNN
 F 1 "Conn_01x08_Male" H 5706 2087 50  0000 C CNN
 F 2 "" H 5600 1700 50  0001 C CNN
@@
 $EndComp
 $Comp
-L Connector:Conn_01x08_Male J?
+L Connector:Conn_01x08_Male J4
 U 1 1 5BFFB07D
 P 4900 1700
-F 0 "J?" H 5006 2178 50  0000 C CNN
+F 0 "J4" H 5006 2178 50  0000 C CNN
 F 1 "Conn_01x08_Male" H 5006 2087 50  0000 C CNN
 F 2 "" H 4900 1700 50  0001 C CNN
@@
 MINI SD CARD \nhttps://learn.adafruit.com/adafruit-micro-sd-breakout-board-card-tutorial/download
 $Comp
-L Device:C C?
+L Device:C C8
 U 1 1 5C01A2F6
 P 3350 4750
-F 0 "C?" H 3465 4796 50  0000 L CNN
+F 0 "C8" H 3465 4796 50  0000 L CNN
 F 1 "1u" H 3465 4705 50  0000 L CNN
 F 2 "" H 3388 4600 50  0001 C CNN
@@
 $EndComp
 $Comp
-L Device:CP C?
+L Device:CP C9
 U 1 1 5C023C80
 P 3750 4750
-F 0 "C?" H 3868 4796 50  0000 L CNN
+F 0 "C9" H 3868 4796 50  0000 L CNN
 F 1 "4.7u" H 3868 4705 50  0000 L CNN
 F 2 "" H 3788 4600 50  0001 C CNN
@@
 	550  3300 550  7650
 $Comp
-L Regulator_Linear:LP2985-3.3 U?
+L Regulator_Linear:LP2985-3.3 U5
 U 1 1 5C075051
 P 6050 3900
-F 0 "U?" H 6050 4242 50  0000 C CNN
+F 0 "U5" H 6050 4242 50  0000 C CNN
 F 1 "LP2985-3.3" H 6050 4151 50  0000 C CNN
 F 2 "Package_TO_SOT_SMD:SOT-23-5" H 6050 4225 50  0001 C CNN
@@
 $EndComp
 $Comp
-L power:+3V3 #PWR?
+L power:+3V3 #PWR020
 U 1 1 5C0753B8
 P 6550 3750
-F 0 "#PWR?" H 6550 3600 50  0001 C CNN
+F 0 "#PWR020" H 6550 3600 50  0001 C CNN
 F 1 "+3V3" H 6565 3923 50  0000 C CNN
 F 2 "" H 6550 3750 50  0001 C CNN
@@
 	6550 3800 6550 3750
 $Comp
-L power:GND #PWR?
+L power:GND #PWR018
 U 1 1 5C0774A6
 P 6050 4200
-F 0 "#PWR?" H 6050 3950 50  0001 C CNN
+F 0 "#PWR018" H 6050 3950 50  0001 C CNN
 F 1 "GND" H 6055 4027 50  0000 C CNN
 F 2 "" H 6050 4200 50  0001 C CNN
@@
 $EndComp
 $Comp
-L power:+5V #PWR?
+L power:+5V #PWR017
 U 1 1 5C0779E3
 P 5550 3800
-F 0 "#PWR?" H 5550 3650 50  0001 C CNN
+F 0 "#PWR017" H 5550 3650 50  0001 C CNN
 F 1 "+5V" H 5565 3973 50  0000 C CNN
 F 2 "" H 5550 3800 50  0001 C CNN
@@
 	5650 3800 5550 3800
 $Comp
-L Device:C C?
+L Device:C C13
 U 1 1 5C079EC3
 P 6800 3950
-F 0 "C?" H 6915 3996 50  0000 L CNN
+F 0 "C13" H 6915 3996 50  0000 L CNN
 F 1 "100 nF" H 6915 3905 50  0000 L CNN
 F 2 "" H 6838 3800 50  0001 C CNN
@@
 $EndComp
 $Comp
-L Device:C C?
+L Device:C C10
 U 1 1 5C07A03B
 P 5100 3950
-F 0 "C?" H 5215 3996 50  0000 L CNN
+F 0 "C10" H 5215 3996 50  0000 L CNN
 F 1 "100 nF" H 5215 3905 50  0000 L CNN
 F 2 "" H 5138 3800 50  0001 C CNN
@@
 Connection ~ 6550 3800
 $Comp
-L power:GND #PWR?
+L power:GND #PWR016
 U 1 1 5C07E085
 P 5100 4100
-F 0 "#PWR?" H 5100 3850 50  0001 C CNN
+F 0 "#PWR016" H 5100 3850 50  0001 C CNN
 F 1 "GND" H 5105 3927 50  0000 C CNN
 F 2 "" H 5100 4100 50  0001 C CNN
@@
 $EndComp
 $Comp
-L power:GND #PWR?
+L power:GND #PWR022
 U 1 1 5C07E0DA
 P 6800 4100
-F 0 "#PWR?" H 6800 3850 50  0001 C CNN
+F 0 "#PWR022" H 6800 3850 50  0001 C CNN
 F 1 "GND" H 6805 3927 50  0000 C CNN
 F 2 "" H 6800 4100 50  0001 C CNN
@@
 insert CD54HC4050 here (level shifter)
 $Comp
-L Connector:Micro_SD_Card J?
+L Connector:Micro_SD_Card J6
 U 1 1 5C085268
 P 8600 5450
-F 0 "J?" H 8550 6167 50  0000 C CNN
+F 0 "J6" H 8550 6167 50  0000 C CNN
 F 1 "Micro_SD_Card" H 8550 6076 50  0000 C CNN
 F 2 "" H 9750 5750 50  0001 C CNN
@@
 $EndComp
 $Comp
-L power:GND #PWR?
+L power:GND #PWR030
 U 1 1 5C0855B0
 P 9400 6050
-F 0 "#PWR?" H 9400 5800 50  0001 C CNN
+F 0 "#PWR030" H 9400 5800 50  0001 C CNN
 F 1 "GND" H 9405 5877 50  0000 C CNN
 F 2 "" H 9400 6050 50  0001 C CNN
@@
 	7300 5850 7700 5850
 $Comp
-L power:GND #PWR?
+L power:GND #PWR025
 U 1 1 5C0B5CF7
 P 7550 5650
-F 0 "#PWR?" H 7550 5400 50  0001 C CNN
+F 0 "#PWR025" H 7550 5400 50  0001 C CNN
 F 1 "GND" H 7555 5477 50  0000 C CNN
 F 2 "" H 7550 5650 50  0001 C CNN
@@
 $EndComp
 $Comp
-L power:+3V3 #PWR?
+L power:+3V3 #PWR024
 U 1 1 5C0B5E0C
 P 7300 5450
-F 0 "#PWR?" H 7300 5300 50  0001 C CNN
+F 0 "#PWR024" H 7300 5300 50  0001 C CNN
 F 1 "+3V3" H 7315 5623 50  0000 C CNN
 F 2 "" H 7300 5450 50  0001 C CNN
