File: KicadFiles/testbaja.sch (KiCad schematic (older format))
At the start: 11 parts, among them J1 Conn_01x05_Male, J10 Conn_01x02_Female, J2 Conn_01x08_Female, J3 Conn_01x04_Female, J4 Conn_01x04_Female, J5 Conn_01x16_Female, J6 Conn_01x04_Female, J7 Conn_01x04_Female, J8 Conn_01x04_Female, J9 Conn_01x30_Female

Commit message: all file update before i install ubuntu
Parts:
- removed J10: Conn_01x02_Female, symbol Connector:Conn_01x02_Female
- added F1: Fuse, symbol Device:Fuse
- added J10: Conn_01x04_Female, TestBaja:DC_Connector, symbol Connector:Conn_01x04_Female
- gave numbers to parts that had none: 1
Connections:
- net labels added: IN_UNFUSED
- net labels removed: 3v3, CLK
- wire segments 88 -> 93
Changed lines of the file:
@@
 d12
 Text Label 4000 2750 0    50   ~ 0
-CLK
+SCK
 Text Label 4000 2850 0    50   ~ 0
 GND
@@
 GND
 Text Label 5800 1550 0    50   ~ 0
-3v3
+3V3
 Text Label 5800 1650 0    50   ~ 0
 d11
@@
 SCK
 Text Label 8950 2900 0    50   ~ 0
-3v3
+3V3
 Text Label 8950 3000 0    50   ~ 0
 ref
@@
 Text Notes 6350 1650 0    50   ~ 0
 sdi
-$Comp
-L Connector:Conn_01x02_Female J10
-U 1 1 5BB79404
-P 3000 1200
-F 0 "J10" H 3027 1176 50  0000 L CNN
-F 1 "Conn_01x02_Female" H 3027 1085 50  0000 L CNN
-F 2 "" H 3000 1200 50  0001 C CNN
-F 3 "~" H 3000 1200 50  0001 C CNN
-	1    3000 1200
-	1    0    0    -1
-$EndComp
-Wire Wire Line
-	2800 1200 2550 1200
-Wire Wire Line
-	2550 1300 2800 1300
-Text Label 2550 1200 0    50   ~ 0
-IN
-Text Label 2550 1300 0    50   ~ 0
+Text Label 2600 1400 0    50   ~ 0
+IN_UNFUSED
+Text Label 2600 1300 0    50   ~ 0
 GND
 Wire Wire Line
@@
 Connection ~ 6100 2550
 $Comp
-L Device:R R?
+L Device:R R1
 U 1 1 5BB970D7
 P 4150 2200
-F 0 "R?" H 4220 2246 50  0000 L CNN
+F 0 "R1" H 4220 2246 50  0000 L CNN
 F 1 "R" H 4220 2155 50  0000 L CNN
 F 2 "Resistor_SMD:R_1206_3216Metric_Pad1.42x1.75mm_HandSolder" V 4080 2200 50  0001 C CNN
@@
 Text Label 4150 1850 0    50   ~ 0
 5V
+$Comp
+L Device:Fuse F1
+U 1 1 5BBD7D5C
+P 2200 1650
+F 0 "F1" H 2260 1696 50  0000 L CNN
+F 1 "Fuse" H 2260 1605 50  0000 L CNN
+F 2 "" V 2130 1650 50  0001 C CNN
+F 3 "~" H 2200 1650 50  0001 C CNN
+	1    2200 1650
+	1    0    0    -1
+$EndComp
+Wire Wire Line
+	2200 1800 2200 1850
+Wire Wire Line
+	2200 1850 2500 1850
+Text Label 2500 1850 0    50   ~ 0
+IN
+$Comp
+L Connector:Conn_01x04_Female J10
+U 1 1 5BBFF9EB
+P 3300 1300
+F 0 "J10" H 3327 1276 50  0000 L CNN
+F 1 "Conn_01x04_Female" H 3327 1185 50  0000 L CNN
+F 2 "TestBaja:DC_Connector" H 3300 1300 50  0001 C CNN
+F 3 "~" H 3300 1300 50  0001 C CNN
+	1    3300 1300
+	1    0    0    -1
+$EndComp
+Wire Wire Line
+	3100 1300 2600 1300
+Wire Wire Line
+	2200 1400 2200 1500
+Wire Wire Line
+	2200 1400 3100 1400
+Wire Wire Line
+	3100 1500 2600 1500
+Wire Wire Line
+	2600 1200 3100 1200
+Text Label 2600 1200 0    50   ~ 0
+GND
+Text Label 2600 1500 0    50   ~ 0
+GND
 $EndSCHEMATC

Commit message: ORDERED BOARDS
Parts:
- added D1: RED, LED_THT:LED_D5.0mm_FlatTop, symbol LED:CQY99
- added R2: 220, Resistor_SMD:R_0805_2012Metric, symbol Device:R
- F1: footprint (none) -> TestBaja:Fuse_0ZCFSeries
Connections:
- net 5V: no longer J1.2 (Pin_2)
- net GND: now also R2.2
- net IN: now also F1.1, J1.2 (Pin_2), D1.2 (A); no longer F1.2
- net IN_UNFUSED: now also F1.2; no longer F1.1
- new net: D1.1 (K), R2.1
Other:
- moved on the sheet: F1
Changed lines of the file:
@@
 GND
 Wire Wire Line
-	3500 2750 3500 2450
-Wire Wire Line
-	2900 2450 3500 2450
-Wire Wire Line
-	2900 2750 3500 2750
+	2900 2450 3200 2450
 Wire Wire Line
 	6100 2250 6050 2250
@@
 L Device:Fuse F1
 U 1 1 5BBD7D5C
-P 2200 1650
-F 0 "F1" H 2260 1696 50  0000 L CNN
-F 1 "Fuse" H 2260 1605 50  0000 L CNN
-F 2 "" V 2130 1650 50  0001 C CNN
-F 3 "~" H 2200 1650 50  0001 C CNN
-	1    2200 1650
-	1    0    0    -1
+P 2050 1400
+F 0 "F1" H 2110 1446 50  0000 L CNN
+F 1 "Fuse" H 2110 1355 50  0000 L CNN
+F 2 "TestBaja:Fuse_0ZCFSeries" V 1980 1400 50  0001 C CNN
+F 3 "~" H 2050 1400 50  0001 C CNN
+	1    2050 1400
+	0    -1   -1   0
 $EndComp
-Wire Wire Line
-	2200 1800 2200 1850
-Wire Wire Line
-	2200 1850 2500 1850
-Text Label 2500 1850 0    50   ~ 0
+Text Label 1800 1400 0    50   ~ 0
 IN
 $Comp
@@
 	3100 1300 2600 1300
 Wire Wire Line
-	2200 1400 2200 1500
-Wire Wire Line
 	2200 1400 3100 1400
 Wire Wire Line
@@
 Text Label 2600 1500 0    50   ~ 0
 GND
+$Comp
+L LED:CQY99 D1
+U 1 1 5BC89853
+P 1650 1550
+F 0 "D1" V 1646 1472 50  0000 R CNN
+F 1 "RED" V 1555 1472 50  0000 R CNN
+F 2 "LED_THT:LED_D5.0mm_FlatTop" H 1650 1725 50  0001 C CNN
+F 3 "https://www.prtice.info/IMG/pdf/CQY99.pdf" H 1600 1550 50  0001 C CNN
+	1    1650 1550
+	0    -1   -1   0
+$EndComp
+$Comp
+L Device:R R2
+U 1 1 5BC8CD5C
+P 1650 1900
+F 0 "R2" H 1720 1946 50  0000 L CNN
+F 1 "220" H 1720 1855 50  0000 L CNN
+F 2 "Resistor_SMD:R_0805_2012Metric" V 1580 1900 50  0001 C CNN
+F 3 "~" H 1650 1900 50  0001 C CNN
+	1    1650 1900
+	1    0    0    -1
+$EndComp
+Wire Wire Line
+	1650 2050 1650 2100
+Wire Wire Line
+	1650 2100 1950 2100
+Text Label 1950 2100 0    50   ~ 0
+GND
+Wire Wire Line
+	1650 1400 1650 1450
+Wire Wire Line
+	1650 1400 1900 1400
+Wire Wire Line
+	3200 2550 3200 2450
+Wire Wire Line
+	2900 2750 3200 2750
 $EndSCHEMATC

Commit message: Fixed frontdash can CS
Connections:
- net CS is gone; now on net d10: J5.6 (Pin_6)
Changed lines of the file:
@@
 EESchema Schematic File Version 4
-LIBS:testbaja-cache
-EELAYER 26 0
+EELAYER 28 0
 EELAYER END
 $Descr A4 11693 8268
@@
 SCK
 Text Label 5800 1950 0    50   ~ 0
-CS
+d10
 Text Label 5800 2050 0    50   ~ 0
 RST
