File: KicadFiles/Backdash_v1.5/backdash/backdash_v1.5.kicad_pcb (KiCad board)
At the start: 2 copper layers, 96.5 x 68.6 mm, 23 parts, among them Q1 2N3904

Commit message: gerbers exist now
Routing:
- net /GND: vias 162 -> 183
Other:
- board text added: "Backdash_v1.5 / 2019 - Magic Squad"
- board text removed: "Backdash_v1.5 / 2019 - Skye Ozga"
Changed lines of the file:
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@@
     (thickness 1.6)
     (drawings 9)
-    (tracks 305)
+    (tracks 326)
     (zones 0)
     (modules 23)
@@
       (xy -6.702229 -4.977358) (xy -6.486088 -5.005262) (xy -6.326909 -5.018797) (xy -5.80409 -5.016603)) (layer F.SilkS) (width 0.01))
   )
-  (gr_text "Backdash_v1.5 / 2019\n- Skye Ozga" (at 147.32 59.69) (layer F.SilkS)
+  (gr_text "Backdash_v1.5 / 2019\n- Magic Squad" (at 147.32 59.69) (layer F.SilkS)
     (effects (font (size 1 1) (thickness 0.15)))
   )
@@
   (via (at 109.22 77.47) (size 0.8) (drill 0.4) (layers F.Cu B.Cu) (net 1))
   (via (at 111.76 73.66) (size 0.8) (drill 0.4) (layers F.Cu B.Cu) (net 1))
-  (via (at 111.76 52.07) (size 0.8) (drill 0.4) (layers F.Cu B.Cu) (net 1))
+  (via (at 111.76 53.34) (size 0.8) (drill 0.4) (layers F.Cu B.Cu) (net 1))
   (via (at 111.76 33.02) (size 0.8) (drill 0.4) (layers F.Cu B.Cu) (net 1))
   (via (at 109.22 72.39) (size 0.8) (drill 0.4) (layers F.Cu B.Cu) (net 1))
@@
   (via (at 106.68 39.37) (size 0.8) (drill 0.4) (layers F.Cu B.Cu) (net 1))
   (via (at 128.27 82.55) (size 0.8) (drill 0.4) (layers F.Cu B.Cu) (net 1))
+  (via (at 135.89 78.74) (size 0.8) (drill 0.4) (layers F.Cu B.Cu) (net 1))
+  (via (at 135.89 81.28) (size 0.8) (drill 0.4) (layers F.Cu B.Cu) (net 1))
+  (via (at 142.24 81.28) (size 0.8) (drill 0.4) (layers F.Cu B.Cu) (net 1))
+  (via (at 140.97 52.07) (size 0.8) (drill 0.4) (layers F.Cu B.Cu) (net 1))
+  (via (at 116.84 26.67) (size 0.8) (drill 0.4) (layers F.Cu B.Cu) (net 1))
+  (via (at 116.84 24.13) (size 0.8) (drill 0.4) (layers F.Cu B.Cu) (net 1))
+  (via (at 106.68 24.13) (size 0.8) (drill 0.4) (layers F.Cu B.Cu) (net 1))
+  (via (at 101.6 24.13) (size 0.8) (drill 0.4) (layers F.Cu B.Cu) (net 1))
+  (via (at 96.52 24.13) (size 0.8) (drill 0.4) (layers F.Cu B.Cu) (net 1))
+  (via (at 91.44 24.13) (size 0.8) (drill 0.4) (layers F.Cu B.Cu) (net 1))
+  (via (at 86.36 24.13) (size 0.8) (drill 0.4) (layers F.Cu B.Cu) (net 1))
+  (via (at 81.28 24.13) (size 0.8) (drill 0.4) (layers F.Cu B.Cu) (net 1))
+  (via (at 81.28 21.59) (size 0.8) (drill 0.4) (layers F.Cu B.Cu) (net 1))
+  (via (at 86.36 21.59) (size 0.8) (drill 0.4) (layers F.Cu B.Cu) (net 1))
+  (via (at 91.44 21.59) (size 0.8) (drill 0.4) (layers F.Cu B.Cu) (net 1))
+  (via (at 96.52 21.59) (size 0.8) (drill 0.4) (layers F.Cu B.Cu) (net 1))
+  (via (at 101.6 21.59) (size 0.8) (drill 0.4) (layers F.Cu B.Cu) (net 1))
+  (via (at 106.68 21.59) (size 0.8) (drill 0.4) (layers F.Cu B.Cu) (net 1))
+  (via (at 111.76 21.59) (size 0.8) (drill 0.4) (layers F.Cu B.Cu) (net 1))
+  (via (at 74.93 24.13) (size 0.8) (drill 0.4) (layers F.Cu B.Cu) (net 1))
+  (via (at 130.81 20.32) (size 0.8) (drill 0.4) (layers F.Cu B.Cu) (net 1))
   (via (at 97.79 39.37) (size 0.8) (drill 0.4) (layers F.Cu B.Cu) (net 2))
   (segment (start 64.77 27.94) (end 63.5 29.21) (width 0.508) (layer F.Cu) (net 2))

Commit message: labeled nanos
Parts:
- removed G***: LOGO, TestBaja:Baja_Logo_Backdash
- NANO1 // Tach: renamed from NANO1
- NANO2 // Wheel: renamed from NANO2
- NANO3 // CVT: renamed from NANO3

Commit message: oops un-deleted logo
Parts:
- added G***: LOGO, TestBaja:Baja_Logo_Backdash, F.Cu at (147.3, 68.6)
